Commit message: make .rviz file

File: urdf/robot_practice.urdf.xacro (robot description, xacro)
@@ -72,5 +72,5 @@
   </link>
   <joint name="scan_joint" type="fixed">
-    <origin xyz="-0.0017476 -0.332 0.086" rpy="0 0 0" />
+    <origin xyz="-0.0017476 -0.332 0.086" rpy="1.5708 0 0" />
     <parent link="base_link" />
     <child link="base_scan" />
