Commit message: upgrade urdf demo

File: urdf/urdf2.urdf (robot description, URDF)
Before this commit: robot AGV, 10 links, 9 joints
Links:
- link base_link: mass 0.38435995228823 -> 3.83244977936653
- link imu_link: mass 3.64288404677104E-08 -> 3.64288391721299E-08
- link wheel_left_link: mass 0.0496616978661662 -> 0.0496616978661665
- link wheel_right_link: mass 0.0496616978661661 -> 0.0496616978661664
