Commit message: check error

File: urdf/AGV.urdf (robot description, URDF)
Before this commit: robot AGV, 10 links, 9 joints
Links:
- removed link imu_link
- added link camera_link, mass 3.64288404677104E-08; collision mesh filename=package://robot_description/meshes/imu_link.STL; visual mesh filename=package://robot_description/meshes/imu_link.STL
Joints:
- joint imu_joint: child imu_link -> camera_link

Commit message: update 10/03

File: urdf/AGV.urdf (robot description, URDF)
Before this commit: robot AGV, 10 links, 9 joints
Links:
- removed link camera_link
- added link imu_link, mass 0.000289811922293658; collision mesh filename=package://robot_description/meshes/imu_link.STL; visual mesh filename=package://robot_description/meshes/imu_link.STL
- link back_rotate_link: mass 0.023917826288437 -> 0.134968786413858; geometry collision mesh filename=package://robot_description/meshes/back_link.STL; visual mesh filename=package://robot_description/meshes/back_link.STL
- link back_wheel_link: mass 0.0469863288657831 -> 0.192670881607509; geometry collision mesh filename=package://robot_description/meshes/b_wheel_link.STL; visual mesh filename=package://robot_description/meshes/b_wheel_link.STL
- link base_link: mass 0.38435995228823 -> 3.47951537357257
- link base_scan: mass 0.166060934057212 -> 0.166053843630804
- link front_rotate_link: mass 0.023917826288437 -> 0.134968786413858; geometry collision mesh filename=package://robot_description/meshes/front_link.STL; visual mesh filename=package://robot_description/meshes/front_link.STL
- link front_wheel_link: mass 0.0469863288657831 -> 0.192670881607509; geometry collision mesh filename=package://robot_description/meshes/f_wheel_link.STL; visual mesh filename=package://robot_description/meshes/f_wheel_link.STL
- link wheel_left_link: mass 0.0496616978661662 -> 0.0848957004604736
- link wheel_right_link: mass 0.0496616978661661 -> 0.0848957004604734
Joints:
- joint back_rotate_joint: origin xyz=-0.1385 0 -0.00985 rpy=-3.1416 0 -0.20493 -> xyz=-0.122 0.00012091 -0.015 rpy=0 0 0
- joint back_wheel_joint: axis 0 -1 0 -> 0 1 0; origin xyz=0.033 0 0.03635 rpy=0 0 0 -> xyz=-0.019817 0 -0.059 rpy=0 0 0
- joint front_rotate_joint: axis 0 0 1 -> 0 0 -1; origin xyz=0.1385 0 -0.00985 rpy=0 0 1.0273 -> xyz=0.122 -0.00012091 -0.015 rpy=0 0 0
- joint front_wheel_joint: axis 0 -1 0 -> 0 1 0; origin xyz=-0.033 0 -0.03635 rpy=0 0 0 -> xyz=0.019817 0 -0.059 rpy=0 0 0
- joint imu_joint: child camera_link -> imu_link; origin xyz=0.20152 -0.0019616 0.0175 rpy=0 0 0 -> xyz=0 0 0 rpy=0 0 0
- joint scan_joint: origin xyz=0.132 -0.0017476 0.083 rpy=0 0 0 -> xyz=0.132 -0.00013082 0.053 rpy=0 0 0
- joint wheel_left_joint: origin xyz=0 -0.186 -0.0387 rpy=0 0 0 -> xyz=0.00016087 0.16232 -0.0665 rpy=0 0 -0.00099109
- joint wheel_right_joint: origin xyz=0 0.186 -0.0387 rpy=0 0 0 -> xyz=-0.00016087 -0.16232 -0.0665 rpy=0 0 -0.00099109
